Commit message: Feature/aruco bt (#65)
* Added Aruco Marker 0 model

* Fixed model.config

* Added normal camera to URDF

* Add Bounding Box (BB) msg for Aruco detection

* Fixed import path for BB msg

* Added BB to CMakeLists so the interface is generated

* Fixed ArUco marker image, previous one wasn't 4x4 50

* Fixed aruco_node OpenCV version issues, added support for sim parameter

* Changed BB to Detection 2D

* Added ROS gz bridge for camera

* Slightly increase forward speed when aruco isn't detecte

* In progress: Added cpp aruco node that publishes aruco pose in map frame, working on BT stuff

* Fixed aruco pose estimation

* Made aruco goal pose same orientation as rover currently

* Changed info messages to warning

* Added archimedean spiral path coverage

* Cleaned up BT, fixed spiral generation to start at actual rover position, fixed stale aruco pose issue

* Changed default nav mode back to GNSS

* Get rid of old camera

* Fixed sime time vs real time issue, made spiral path start align with current rover orientation

* Changed sim parameter to use_sim_time

* Added GNSS navigation to aruco branch

* Oops forgot to switch default to GNSS

* Added sim transform for rgb camera

* Moved aruco launch to navigation launch

* Removed unnecessary aruco sdfs

File: src/description/urdf/zed_macro_sim.urdf.xacro (robot description, xacro)
@@ -43,4 +43,10 @@
       <child link="${name}_left_camera_frame_optical"/>
     </joint>
+    <link name="athena/base_footprint/${name}_rgb_sensor"/>
+    <joint name="${name}_rgb_sensor_joint" type="fixed">
+      <origin xyz="0 0 0" rpy="-${M_PI/2} 0.0 -${M_PI/2}"/>
+      <parent link="${name}_left_camera_frame"/>
+      <child link="athena/base_footprint/${name}_rgb_sensor"/>
+    </joint>
     <link name="${name}_right_camera_frame" />
     <joint name="${name}_right_camera_joint" type="fixed">
