Commit message: Recovered changes on clean branch

File: src/description/ros2_control/arm/arm.rmd.ros2_control.xacro (robot description, xacro)
@@ -5,5 +5,5 @@
       <hardware>
         <plugin>rmd_ros2_control/RMDHardwareInterface</plugin>
-        <param name="update_rate">2</param> <!-- Hz -->
+        <param name="update_rate">10</param> <!-- Hz -->
         <param name="logger_rate">5</param> <!-- Hz -->
         <param name="logger_state">0</param> <!-- 0 for off, 1 for on -->

File: src/description/ros2_control/arm/arm.servo.ros2_control.xacro (robot description, xacro)
@@ -5,5 +5,5 @@
             <hardware>
                 <plugin>servo_ros2_control/SERVOHardwareInterface</plugin>
-                <param name="update_rate">1</param> <!-- Hz -->
+                <param name="update_rate">10</param> <!-- Hz -->
                 <param name="logger_rate">5</param> <!-- Hz -->
                 <param name="logger_state">0</param> <!-- 0 for off, 1 for on -->

File: src/description/ros2_control/arm/arm.smc.ros2_control.xacro (robot description, xacro)
@@ -5,5 +5,5 @@
       <hardware>
         <plugin>smc_ros2_control/SMCHardwareInterface</plugin>
-        <param name="update_rate">2</param> <!-- Hz -->
+        <param name="update_rate">10</param> <!-- Hz -->
         <param name="logger_rate">5</param> <!-- Hz -->
         <param name="logger_state">0</param> <!-- 0 for off, 1 for on -->
@@ -11,6 +11,6 @@
       </hardware>
       <joint name="base_yaw">
-        <param name="node_id">0x148</param>
-        <param name="gear_ratio">-100</param>
+        <param name="node_id">0x145</param>
+        <param name="gear_ratio">40</param>
         <param name="operating_velocity">300</param> <!-- motor dps -->
         <command_interface name="position"/>
@@ -22,5 +22,5 @@
       </joint>
       <joint name="wrist_pitch">
-        <param name="node_id">0x145</param>
+        <param name="node_id">0x148</param>
         <param name="gear_ratio">40</param>
         <param name="operating_velocity">1000</param> <!-- motor dps -->

File: src/description/ros2_control/science/science.mock.ros2_control.xacro (robot description, xacro)
@@ -48,10 +48,10 @@
                 <state_interface name="velocity"/>
             </joint>
-            <joint name="servo_scoop_a">
+            <joint name="scoop_a">
                 <command_interface name="position"/>
                 <command_interface name="velocity"/>
                 <state_interface name="position"/>
             </joint>
-            <joint name="servo_scoop_b">
+            <joint name="scoop_b">
                 <command_interface name="position"/>
                 <command_interface name="velocity"/>

File: src/description/ros2_control/science/science.servo.ros2_control.xacro (robot description, xacro)
@@ -5,17 +5,11 @@
             <hardware>
                 <plugin>servo_ros2_control/SERVOHardwareInterface</plugin>
-                <param name="update_rate">20</param> <!-- Hz -->
+                <param name="update_rate">10</param> <!-- Hz -->
                 <param name="logger_rate">5</param> <!-- Hz -->
-                <param name="logger_state">1</param> <!-- 0 for off, 1 for on -->
+                <param name="logger_state">0</param> <!-- 0 for off, 1 for on -->
                 <param name="can_interface">can0</param>
                 <param name="can_id">0x80</param>
             </hardware>
-            <joint name="servo_rack_and_pinion_l">
-                <param name="node_id">0x1</param>
-                <param name="gear_ratio">1</param>
-                <param name="max_pos">235</param> <!-- degrees -->
-                <param name ="meters_per_deg">0.00016666666</param> <!-- (TODO) convert motor position in degrees to displacement in meters -->
-                <param name="servo_type">standard</param> <!-- standard or continuous -->
-                <param name="joint_type">revolute</param> <!-- revolute or prismatic -->
+            <joint name="rack_and_pinion_left">
                 <command_interface name="position"/>
                 <command_interface name="velocity"/>
@@ -23,11 +17,5 @@
                 <state_interface name="velocity"/>
             </joint>
-            <joint name="servo_rack_and_pinion_r">
-                <param name="node_id">0x2</param>
-                <param name="gear_ratio">1</param>
-                <param name="max_pos">235</param> <!-- degrees -->
-                <param name ="meters_per_deg">0.00016666666</param> <!-- (TODO) convert motor position in degrees to displacement in meters -->
-                <param name="servo_type">standard</param> <!-- standard or continuous -->
-                <param name="joint_type">revolute</param> <!-- revolute or prismatic -->
+            <joint name="rack_and_pinion_right">
                 <command_interface name="position"/>
                 <command_interface name="velocity"/>
@@ -35,6 +23,6 @@
                 <state_interface name="velocity"/>
             </joint>
-            <joint name="servo_scoop_a">
-                <param name="node_id">0x3</param> <!-- 0x5 -->
+            <joint name="scoop_a">
+                <param name="node_id">0x2</param>
                 <param name="gear_ratio">1</param>
                 <param name="max_pos">178</param> <!-- degrees -->
@@ -45,6 +33,6 @@
                 <state_interface name="position"/>
             </joint>
-            <joint name="servo_scoop_b">
-                <param name="node_id">0x5</param> <!-- 0x3 -->
+            <joint name="scoop_b">
+                <param name="node_id">0x3</param>
                 <param name="gear_ratio">1</param>
                 <param name="max_pos">178</param> <!-- degrees -->
@@ -55,11 +43,11 @@
                 <state_interface name="position"/>
             </joint>
-            <joint name="servo_sampler_lift_l">
-                <param name="node_id">0x6</param>
+            <joint name="auger">
+                <param name="node_id">0x4</param>
                 <param name="gear_ratio">1</param>
-                <param name="max_pos">360</param> <!-- degrees -->
+                <param name="max_pos">90</param> <!-- degrees -->
                 <param name ="meters_per_deg">0.00016666666</param> <!-- (TODO) convert motor position in degrees to displacement in meters -->
                 <param name="servo_type">standard</param> <!-- standard / continuous -->
-                <param name="joint_type">revolute</param> <!-- revolute / prismatic -->
+                <param name="joint_type">prismatic</param> <!-- revolute / prismatic -->
                 <command_interface name="position"/>
                 <command_interface name="velocity"/>
@@ -67,23 +55,11 @@
                 <state_interface name="velocity"/>
             </joint>
-            <joint name="servo_sampler_lift_r">
-                <param name="node_id">0x4</param>
-                <param name="gear_ratio">1</param>
-                <param name="max_pos">360</param> <!-- degrees -->
-                <param name ="meters_per_deg">0.00016666666</param> <!-- (TODO) convert motor position in degrees to displacement in meters -->
-                <param name="servo_type">standard</param> <!-- standard / continuous -->
-                <param name="joint_type">revolute</param> <!-- revolute / prismatic -->
-                <command_interface name="position"/>
-                <command_interface name="velocity"/>
-                <state_interface name="position"/>
-                <state_interface name="velocity"/>
-            </joint>
-            <joint name="servo_auger_lift">
-                <param name="node_id">0x0</param>
+            <joint name="cap">
+                <param name="node_id">0x5</param>
                 <param name="gear_ratio">1</param>
                 <param name="max_pos">270</param> <!-- degrees -->
                 <param name ="meters_per_deg">0.00016666666</param> <!-- (TODO) convert motor position in degrees to displacement in meters -->
                 <param name="servo_type">standard</param> <!-- standard / continuous -->
-                <param name="joint_type">revolute</param> <!-- revolute / prismatic -->
+                <param name="joint_type">prismatic</param> <!-- revolute / prismatic -->
                 <command_interface name="position"/>
                 <command_interface name="velocity"/>

File: src/description/ros2_control/science/science.talon.ros2_control.xacro (robot description, xacro)
@@ -10,10 +10,10 @@
         <param name="can_interface">can0</param>
       </hardware>
-      <joint name="talon_auger">
-        <param name="node_id">2</param>
+      <joint name="talon_lift">
+        <param name="node_id">1</param>
         <param name="joint_type">revolute</param>
-        <!-- Motor config (goBilda Saturn 5303 Series 360 RPM) -->
-        <param name="encoder_resolution">1425.1</param>
-        <param name="gear_ratio">50.9</param>
+        <!-- Motor config (Pololu 37D defaults) -->
+        <param name="encoder_resolution">64.0</param>
+        <param name="gear_ratio">102.08</param>
         <param name="inverted">true</param>
         <param name="sensor_phase">true</param>
@@ -30,5 +30,5 @@
       </joint>
       <joint name="talon_scoop">
-        <param name="node_id">0</param>
+        <param name="node_id">2</param>
         <param name="joint_type">revolute</param>
         <!-- Motor config (Pololu 37D defaults) -->

File: src/description/urdf/athena_arm.urdf.xacro (robot description, xacro)
@@ -32,17 +32,5 @@
   <xacro:unless value="$(arg use_mock_hardware)"> <!-- HARDWARE -->
     <xacro:smc_ros2_control name="smc"/>
-    <ros2_control name="talon_mock" type="system">
-      <hardware>
-        <plugin>mock_components/GenericSystem</plugin>
-      </hardware>
-      <joint name="gripper_claw">
-        <command_interface name="position"/>
-        <command_interface name="velocity"/>
-        <state_interface name="position">
-          <param name="initial_value">-0.0</param>
-        </state_interface>
-        <state_interface name="velocity"/>
-      </joint>
-    </ros2_control>
+    <xacro:talon_ros2_control name="talon"/>
     <xacro:rmd_ros2_control name="rmd"/>
     <xacro:servo_ros2_control name="servo"/>
