Commit message: New 3 dof setup (#108)
* configured for a 3dof controller, we can improve base design later

* extra fixes before actual testing

* Update with real life testing code (#78)

* update to latest

* update rear ackermann controller

* Removed bad paramters

* remove todo nodes

* Flipped the turning

* swap the right and left speed

* working on rover

* updated athena_drive.launch.py

* updated zed launch

* maybe fix the zed issue

* updated drive urdf

* ackermann guarding

* teleop config testing

* Added steering limits

* Revert ZED-related changes from nav_testing_2324

Restores upstream/main versions of:
- sensors.launch.py (publish_odom/map defaults, gps_launch)
- zed.launch.py (publish_tf/publish_map_tf back to LaunchConfiguration)
- zed_macro_sim.urdf.xacro (color + rgb_sensor link/joint)
- athena_drive.urdf.xacro (unconditional zed include + original origin)
- nav_bringup.launch.py (remove zed_to_base_footprint static tf)

* added arm bringup files

* bring over arm can id update as well

---------

Co-authored-by: Adrian Cires <ciresadrian@hotmail.com>
Co-authored-by: UMDLoop Jetson Orin NX <umdloop@gmail.com>

* working, but code wise it should not be prismatic, suitable for now

* allows the user to deactivate the talons and have a mock hardware replacement for just those joints

* Separates arm into 3 subsections, arm, wrist, and end effector due to the individuality and interchangeability of each subsection. This commit has a separate joint by joint controller for arm (composed of base_yaw, shoulder_pitch, and elbow_pitch), 3 wrist controllers (joint by joint for 3dof, 2dof, and an orientation controller for 3DOF), and gripper claw. If we ever decide to add more joints to arm, use a different kind of wrist control scheme, or have a different kind of end effector entirely, the components as well as the code can now be swapped in and out for it.

* Realized a lot of controller switcher functionality had to be modified, so it now functions with this arm setup (will require considerations of drive and always active controllers in yaml file). Also made a 2dof and 3dof trajectory controller config.

---------

Co-authored-by: Mohammad Durrani <46766905+mdurrani808@users.noreply.github.com>
Co-authored-by: Adrian Cires <ciresadrian@hotmail.com>
Co-authored-by: UMDLoop Jetson Orin NX <umdloop@gmail.com>
Co-authored-by: duttaishan01 <duttaishan01@FIGARO.myguest.virtualbox.org>

File: src/description/ros2_control/arm/arm.smc_2dof.ros2_control.xacro (robot description, xacro)
@@ -1,5 +1,5 @@
 <?xml version="1.0"?>
 <robot xmlns:xacro="http://www.ros.org/wiki/xacro">
-  <xacro:macro name="smc_ros2_control" params="name">
+  <xacro:macro name="smc_2dof_ros2_control" params="name">
     <ros2_control name="${name}" type="system">
       <hardware>

File: src/description/ros2_control/arm/arm.talon_2dof.ros2_control.xacro (robot description, xacro)
@@ -1,15 +1,21 @@
 <?xml version="1.0"?>
 <robot xmlns:xacro="http://www.ros.org/wiki/xacro">
-  <xacro:macro name="talon_ros2_control" params="name">
+  <xacro:macro name="talon_2dof_ros2_control" params="name deactivate_talon">
     <ros2_control name="${name}" type="system">
       <hardware>
-        <plugin>talon_ros2_control/TALONHardwareInterface</plugin>
-        <param name="update_rate">10</param> <!-- Hz -->
-        <param name="logger_rate">5</param> <!-- Hz -->
-        <param name="logger_state">0</param> <!-- 0 for off, 1 for on -->
-        <param name="can_interface">can0</param>
+        <param name="deactivate_talon">${deactivate_talon}</param>
+        <xacro:if value="${deactivate_talon}">
+          <plugin>mock_components/GenericSystem</plugin>
+        </xacro:if>
+        <xacro:unless value="${deactivate_talon}">
+          <plugin>talon_ros2_control/TALONHardwareInterface</plugin>
+          <param name="update_rate">10</param> <!-- Hz -->
+          <param name="logger_rate">5</param> <!-- Hz -->
+          <param name="logger_state">0</param> <!-- 0 for off, 1 for on -->
+          <param name="can_interface">can0</param>
+        </xacro:unless>
       </hardware>
       <joint name="gripper_claw">
-        <param name="node_id">2</param>
+        <param name="node_id">4</param>
         <param name="max_disp">0.06</param> <!-- meters -->
         <param name="joint_type">prismatic</param>

File: src/description/ros2_control/drive/drive.rmd.ros2_control.xacro (robot description, xacro)
@@ -5,5 +5,5 @@
       <hardware>
         <plugin>rmd_ros2_control/RMDHardwareInterface</plugin>
-        <param name="update_rate">10</param> <!-- Hz -->
+        <param name="update_rate">30</param> <!-- Hz -->
         <param name="logger_rate">5</param> <!-- Hz -->
         <param name="logger_state">0</param> <!-- 0 for off, 1 for on -->

File: src/description/ros2_control/science/science.talon.ros2_control.xacro (robot description, xacro)
@@ -1,12 +1,18 @@
 <?xml version="1.0"?>
 <robot xmlns:xacro="http://www.ros.org/wiki/xacro">
-  <xacro:macro name="talon_ros2_control" params="name">
+  <xacro:macro name="talon_ros2_control" params="name deactivate_talon">
     <ros2_control name="${name}" type="system">
       <hardware>
-        <plugin>talon_ros2_control/TALONHardwareInterface</plugin>
-        <param name="update_rate">10</param> <!-- Hz -->
-        <param name="logger_rate">5</param> <!-- Hz -->
-        <param name="logger_state">0</param> <!-- 0 for off, 1 for on -->
-        <param name="can_interface">can0</param>
+        <param name="deactivate_talon">${deactivate_talon}</param>
+        <xacro:if value="${deactivate_talon}">
+          <plugin>mock_components/GenericSystem</plugin>
+        </xacro:if>
+        <xacro:unless value="${deactivate_talon}">
+          <plugin>talon_ros2_control/TALONHardwareInterface</plugin>
+          <param name="update_rate">10</param> <!-- Hz -->
+          <param name="logger_rate">5</param> <!-- Hz -->
+          <param name="logger_state">0</param> <!-- 0 for off, 1 for on -->
+          <param name="can_interface">can0</param>
+        </xacro:unless>
       </hardware>
       <joint name="talon_auger">

File: src/description/urdf/athena_arm.urdf.xacro (robot description, xacro)
@@ -8,4 +8,6 @@
   <xacro:arg name="sim_gazebo" default="true"/>
   <xacro:arg name="simulation_controllers" default=""/>
+  <xacro:arg name="use_3dof" default="false"/>
+  <xacro:arg name="deactivate_talon" default="false"/>
   <!-- Macro Imports -->
   <!-- Import athena_arm macro -->
@@ -14,7 +16,9 @@
   <xacro:include filename="$(find description)/config/mock.ros2_control.xacro" />
   <!-- Import smc ros2_control description -->
-  <xacro:include filename="$(find description)/ros2_control/arm/arm.smc.ros2_control.xacro" />
+  <xacro:include filename="$(find description)/ros2_control/arm/arm.smc_2dof.ros2_control.xacro" />
+  <xacro:include filename="$(find description)/ros2_control/arm/arm.smc_3dof.ros2_control.xacro" />
   <!-- Import talon ros2_control description -->
-  <xacro:include filename="$(find description)/ros2_control/arm/arm.talon.ros2_control.xacro" />
+  <xacro:include filename="$(find description)/ros2_control/arm/arm.talon_2dof.ros2_control.xacro" />
+  <xacro:include filename="$(find description)/ros2_control/arm/arm.talon_3dof.ros2_control.xacro" />
   <!-- Import rmd ros2_control description -->
   <xacro:include filename="$(find description)/ros2_control/arm/arm.rmd.ros2_control.xacro" />
@@ -31,18 +35,12 @@
   </xacro:if>
   <xacro:unless value="$(arg use_mock_hardware)"> <!-- HARDWARE -->
-    <xacro:smc_ros2_control name="smc"/>
-    <ros2_control name="talon_mock" type="system">
-      <hardware>
-        <plugin>mock_components/GenericSystem</plugin>
-      </hardware>
-      <joint name="gripper_claw">
-        <command_interface name="position"/>
-        <command_interface name="velocity"/>
-        <state_interface name="position">
-          <param name="initial_value">-0.0</param>
-        </state_interface>
-        <state_interface name="velocity"/>
-      </joint>
-    </ros2_control>
+    <xacro:if value="$(arg use_3dof)">
+      <xacro:talon_3dof_ros2_control name="talon" deactivate_talon="$(arg deactivate_talon)"/>
+      <xacro:smc_3dof_ros2_control name="smc"/>
+    </xacro:if>
+    <xacro:unless value="$(arg use_3dof)">
+      <xacro:talon_2dof_ros2_control name="talon" deactivate_talon="$(arg deactivate_talon)"/>
+      <xacro:smc_2dof_ros2_control name="smc"/>
+    </xacro:unless>
     <xacro:rmd_ros2_control name="rmd"/>
     <xacro:servo_ros2_control name="servo"/>

File: src/description/urdf/athena_science.urdf.xacro (robot description, xacro)
@@ -3,4 +3,5 @@
   <xacro:arg name="use_mock_hardware" default="false"/>
   <xacro:arg name="mock_sensor_commands" default="false"/>
+  <xacro:arg name="deactivate_talon" default="false"/>
   <xacro:include filename="$(find description)/ros2_control/science/science.mock.ros2_control.xacro"/>
   <xacro:include filename="$(find description)/ros2_control/science/science.stepper.ros2_control.xacro" />
@@ -22,5 +23,5 @@
     <xacro:servo_ros2_control name="servo"/>
     <!-- Import talon ros2_control description -->
-    <xacro:talon_ros2_control name="talon"/>
+    <xacro:talon_ros2_control name="talon" deactivate_talon="$(arg deactivate_talon)"/>
     <!-- Import laser ros2_control description (CAN-based) -->
     <xacro:laser_ros2_control name="spectrometry_laser"/>
